Commit message: Update sim2sim

File: resources/robots/titatit/urdf/wheeled_titatit_rl.urdf (robot description, URDF)
Before this commit: robot wheeled_titatit_description, 19 links, 18 joints
Links:
- link FL_foot: geometry collision cylinder length=0.02 radius=0.0948; visual mesh filename=../meshes/FL_foot.STL
- link FR_foot: geometry collision cylinder length=0.02 radius=0.0948; visual mesh filename=../meshes/FR_foot.STL
- link RL_foot: geometry collision cylinder length=0.02 radius=0.0948; visual mesh filename=../meshes/RL_foot.STL
- link RR_foot: geometry collision cylinder length=0.02 radius=0.0948; visual mesh filename=../meshes/RR_foot.STL
